Commit message: downgrade Spinal firmware to use TTL2DXIF

File: robots/gimbalrotor/robots/tri_omni/gimbalrotor.urdf.xacro (robot description, xacro)
@@ -5,6 +5,8 @@
   <xacro:include filename="$(find gimbalrotor)/urdf/tri_omni/common.xacro" />
   <xacro:gimbalrotor_center_link child1="1" child2="2" child3="3"/>
-  <xacro:gimbalrotor_thrust_link self="1" rotor_direction="1"/>
-  <xacro:gimbalrotor_thrust_link self="2" rotor_direction="-1"/>
-  <xacro:gimbalrotor_thrust_link self="3" rotor_direction="1"/>
+  <xacro:gimbalrotor_gimbal_link self="1" rotor_direction="1"/>
+  <xacro:gimbalrotor_gimbal_link self="2" rotor_direction="-1"/>
+  <xacro:gimbalrotor_gimbal_link self="3" rotor_direction="-1"/>
+  <xacro:gimbalrotor_head_link/>
+  <xacro:gimbalrotor_tail_link/>
 </robot>

File: robots/gimbalrotor/urdf/tri_omni/gimbalrotor.urdf.xacro (robot description, xacro)
@@ -23,20 +23,20 @@
     <link name="base_link">
       <inertial>
-        <origin xyz="-0.082255 0.000157 0.014372" rpy="0 0 0"/>
-        <mass value="1.076"/>
-        <inertia
-            ixx="0.005338" iyy="0.006510" izz="0.01052"
-            ixy="0.00000" ixz="0.0000" iyz="0.00000"/>
-      </inertial>
-      <visual>
-        <origin xyz="0 0 0" rpy="0 0 0"/>
-        <geometry>
-          <mesh filename="package://gimbalrotor/urdf/tri/mesh/trirotor_base_link.dae" scale="0.001 0.001 0.001"/>
+        <origin xyz="0.2237 0.0050 0.0126" rpy="0 0 0"/>
+        <mass value="0.74"/>
+        <inertia
+            ixx="0.0011933" iyy="0.0157954" izz="0.0157066"
+            ixy="-0.0008036" ixz="0.0002441" iyz="0.0000132"/>
+      </inertial>
+      <visual>
+        <origin xyz="0 0 0" rpy="0 0 0"/>
+        <geometry>
+          <mesh filename="package://gimbalrotor/urdf/tri_omni/mesh/main_link.dae" scale="0.001 0.001 0.001"/>
         </geometry>
       </visual>
       <collision>
-        <origin xyz="0 0 0" rpy="0 0 0"/>
-        <geometry>
-          <box size="0.234 0.3 0.1"/>
+        <origin xyz="0.2 0 0" rpy="0 0 0"/>
+        <geometry>
+          <box size="0.4 0.3 0.222"/>
         </geometry>
       </collision>
@@ -56,5 +56,5 @@
       <child link="fc"/>
       <parent link="base_link"/>
-      <origin rpy="0 0 0" xyz="0 0 0"/>
+      <origin rpy="0 0 0" xyz="0.33 0 0.067"/>
       <axis xyz="0 0 1"/>
     </joint>
@@ -73,5 +73,5 @@
       <parent link="base_link"/>
       <child link="rotor_arm${child1}"/>
-      <origin rpy="0 0 ${-pi/2}" xyz="0 -0.154 0.051"/>
+      <origin rpy="0 0 ${pi/2}" xyz="0.329 0.065 0.018"/>
       <axis xyz="0 0 1"/>
     </joint>
@@ -89,5 +89,5 @@
       <parent link="base_link"/>
       <child link="rotor_arm${child2}"/>
-      <origin rpy="0 0 ${pi/2}" xyz="0 0.154 0.051"/>
+      <origin rpy="0 0 ${-pi/2}" xyz="0.329 -0.065 0.018"/>
       <axis xyz="0 0 1"/>
     </joint>
@@ -103,65 +103,159 @@
     </link>
     <joint name="base_arm_joint${child3}" type="fixed">
-      <parent link="base_link"/>
+      <parent link="tail_link"/>
       <child link="rotor_arm${child3}"/>
-      <origin rpy="0 0 ${pi}" xyz="-0.214 0 0.051"/>
-      <axis xyz="0 0 1"/>
-    </joint>
-    <xacro:friction self="base_link"/>
-  </xacro:macro>
-  <xacro:macro name="gimbalrotor_thrust_link" params="self rotor_direction">
-    ## link
-    #### gimbal link (roll) ####
-    <link name="gimbal_link_roll${self}">
-      <inertial>
-        <origin xyz="0.076255 0 0" rpy="0 0 0"/>
-        <mass value="0.07"/>
-        <inertia
-            ixx="0.00015" iyy="0.00008" izz="0.00019"
-            ixy="0.0000" ixz="-0.0000" iyz="0.00000"/>
-      </inertial>
-      <!-- <collision> -->
-      <!--   <origin xyz="0.076255 0 0" rpy="0 0 0"/> -->
-      <!--   <geometry> -->
-      <!--     <cylinder radius="0.1" length="0.1"/> -->
-      <!--   </geometry> -->
-      <!-- </collision> -->
-    </link>
-    <xacro:damping_factor link="gimbal_link_roll${self}"/>
-    #### gimbal link (pitch) ####
-    <link name="gimbal_link_pitch${self}">
-      <inertial>
-        <origin xyz="0.076255 0 0" rpy="0 0 0"/>
-        <mass value="0.07"/>
-        <inertia
-            ixx="0.00015" iyy="0.00008" izz="0.00019"
-            ixy="0.0000" ixz="-0.0000" iyz="0.00000"/>
-      </inertial>
-      <collision>
-        <origin xyz="0.076255 0 0" rpy="0 0 0"/>
-        <geometry>
-          <cylinder radius="0.1" length="0.1"/>
-        </geometry>
-      </collision>
+      <origin rpy="0 0 0" xyz="0.076 0 0.0145"/>
+      <axis xyz="0 0 1"/>
+    </joint>
+   <xacro:friction self="base_link"/>
+  </xacro:macro>
+  <xacro:macro name="gimbalrotor_head_link">
+    <!-- head -->
+    <link name="head_link">
+      <inertial>
+        <origin xyz="0.007 0 -0.038" rpy="0 0 0"/>
+        <mass value="0.081"/>
+        <inertia
+            ixx="0.00022881" iyy="0.00022121" izz="0.0"
+            ixy="0.0" ixz="0.00002107" iyz="0.00000009"/>
+      </inertial>
+      <visual>
+        <origin xyz="0 0 0" rpy="0 0 0"/>
+        <geometry>
+          <mesh filename="package://gimbalrotor/urdf/tri_omni/mesh/head_link.dae" scale="0.001 0.001 0.001"/>
+        </geometry>
+      </visual>
+    </link>
+    <xacro:damping_factor link="head_link"/>
+    <joint name="head_joint" type="revolute">
+      <limit effort="6.6" lower="-3.14" upper="3.14" velocity="3.0"/>
+      <parent link="base_link"/>
+      <child link="head_link"/>
+      <origin rpy="0 0 0" xyz="0.41 0 0.018"/>
+      <axis xyz="0 0 1"/>
+      <dynamics damping="0.8" friction="0.0"/>
+    </joint>
+    <transmission name="head_joint_tran">
+      <type>transmission_interface/SimpleTransmission</type>
+      <joint name="head_joint">
+        <hardwareInterface>hardware_interface/EffortJointInterface</hardwareInterface>
+      </joint>
+      <actuator name="head_servo">
+        <hardwareInterface>hardware_interface/EffortJointInterface</hardwareInterface>
+        <mechanicalReduction>1</mechanicalReduction>
+      </actuator>
+    </transmission>
+  </xacro:macro>
+  <xacro:macro name="gimbalrotor_tail_link">
+    <!-- tail -->
+    <link name="tail_link">
+      <inertial>
+        <origin xyz="0.0356 -0.00294 0.00267" rpy="0 0 0"/>
+        <mass value="0.1212457"/>
+        <inertia
+            ixx="0.0000575" ixy="0.0000127" ixz="0.0000036"
+            iyy="0.0000946" iyz="0.0000010"
+            izz="0.0001120"/>
+      </inertial>
+      <visual>
+        <origin xyz="0 0 0" rpy="0 0 0"/>
+        <geometry>
+          <mesh filename="package://gimbalrotor/urdf/tri_omni/mesh/tail_link.dae" scale="1 1 1"/>
+        </geometry>
+      </visual>
+    </link>
+    <xacro:damping_factor link="tail_link"/>
+    <joint name="tail_joint" type="revolute">
+      <limit effort="6.6" lower="-1.57" upper="1.57" velocity="3.0"/>
+      <parent link="base_link"/>
+      <child link="tail_link"/>
+      <origin rpy="0 0 ${pi}" xyz="-0.02 0 0.018"/>
+      <axis xyz="0 1 0"/>
+      <dynamics damping="0.8" friction="0.0"/>
+    </joint>
+    <transmission name="tail_joint_tran">
+      <type>transmission_interface/SimpleTransmission</type>
+      <joint name="tail_joint">
+        <hardwareInterface>hardware_interface/EffortJointInterface</hardwareInterface>
+      </joint>
+      <actuator name="tail_servo">
+        <hardwareInterface>hardware_interface/EffortJointInterface</hardwareInterface>
+        <mechanicalReduction>1</mechanicalReduction>
+      </actuator>
+    </transmission>
+  </xacro:macro>
+  <xacro:macro name="gimbalrotor_gimbal_link" params="self rotor_direction">
+    #### gimbal joints ####
+    <joint name="gimbal${self}_roll" type="revolute">
+      <limit effort="6.6" lower="-2.0" upper="2.0" velocity="3.0"/>
+      <parent link="rotor_arm${self}"/>
+      <child link="gimbal_link${self}"/>
+      <origin rpy="0 0 0" xyz="0 0 0"/>
+      <axis xyz="1 0 0"/>
+      <dynamics damping="0.8" friction="0.0"/>
+    </joint>
+    <transmission name="joint_tran${2*self-1}">
+      <type>transmission_interface/SimpleTransmission</type>
+      <joint name="gimbal${self}_roll">
+        <hardwareInterface>hardware_interface/EffortJointInterface</hardwareInterface>
+      </joint>
+      <actuator name="servo${2*self-1}">
+        <hardwareInterface>hardware_interface/EffortJointInterface</hardwareInterface>
+        <mechanicalReduction>1</mechanicalReduction>
+      </actuator>
+    </transmission>
+    #### gimbal link  ####
+    <link name="gimbal_link${self}">
+      <inertial>
+       <origin xyz="0.074 0.044 0.0" rpy="0 0 0"/>
+        <mass value="0.124"/>
+        <inertia
+            ixx="0.00080131" iyy="0.00021920" izz="0.00099608"
+            ixy="0.00012557" ixz="0.00000026" iyz="-0.00000061"/>
+      </inertial>
+      <visual>
+        <origin xyz="0 0 0" rpy="0 0 0"/>
+        <geometry>
+          <mesh filename="package://gimbalrotor/urdf/tri_omni/mesh/gimbal_link.dae" scale="1 1 1"/>
+        </geometry>
+      </visual>
+    </link>
+    <xacro:damping_factor link="gimbal_link${self}"/>
+    #### rotor joint  ####
+    <joint name="gimbal${self}_pitch" type="revolute">
+      <limit effort="6.6" lower="-2.0" upper="2.0" velocity="3.0"/>
+      <parent link="gimbal_link${self}"/>
+      <child link="rotor_parent${self}"/>
+      <origin rpy="0 0 0" xyz="0.112 0.0877 0"/>
+      <axis xyz="0 1 0"/>
+    </joint>
+    <transmission name="joint_tran${2*self}">
+      <type>transmission_interface/SimpleTransmission</type>
+      <joint name="gimbal${self}_pitch">
+        <hardwareInterface>hardware_interface/EffortJointInterface</hardwareInterface>
+      </joint>
+      <actuator name="servo${2*self}">
+        <hardwareInterface>hardware_interface/EffortJointInterface</hardwareInterface>
+        <mechanicalReduction>1</mechanicalReduction>
+      </actuator>
+    </transmission>
+    ## rotor parent link
+    <link name="rotor_parent${self}">
+      <inertial>
+        <origin xyz="0.09 0 0" rpy="0 0 ${-pi/2}"/>
+        <mass value="0.220"/>
+        <inertia
+            ixx="0.0002011" ixy="0.0000001" ixz="0.0000003"
+            iyy="0.0004337" iyz="0.0"
+            izz="0.0005261"/>
+      </inertial>
       <visual>
         <origin xyz="0 0 0" rpy="0 0 ${-pi/2}"/>
         <geometry>
-          <mesh filename="package://gimbalrotor/urdf/tri/mesh/thrust_link_left_straight.dae" scale="0.001 0.001 0.001"/>
-        </geometry>
-      </visual>
-    </link>
-    <xacro:damping_factor link="gimbal_link_pitch${self}"/>
-    ## rotor parent link (virtual)
-    <link name="rotor_parent${self}">
-      <inertial>
-        <origin xyz="0 0 0" rpy="0 0 0"/>
-        <mass value="0.00001"/>
-        <inertia
-            ixx="0.000001" ixy="0.0" ixz="0.0"
-            iyy="0.000001" iyz="0.0"
-            izz="0.000001"/>
-      </inertial>
-    </link>
-    ## thrust link (virtual)
+          <mesh filename="package://gimbalrotor/urdf/tri_omni/mesh/rotor_link_CW.dae" scale="1 1 1"/>
+        </geometry>
+      </visual>
+    </link>
+    ## thrust link
     <link name="thrust${self}">
       <inertial>
@@ -173,52 +267,12 @@
             izz="0.001"/>
       </inertial>
+      <collision>
+        <origin xyz="0 0 0" rpy="0 0 0"/>
+        <geometry>
+          <cylinder radius="0.1" length="0.1"/>
+        </geometry>
+      </collision>
     </link>
     <xacro:damping_factor link="thrust${self}"/>
-    #### joints ####
-    #### gimbal joint (roll) ####
-    <joint name="gimbal${self}_roll" type="revolute">
-      <limit effort="6.6" lower="-2.0" upper="2.0" velocity="3.0"/>
-      <parent link="rotor_arm${self}"/>
-      <child link="gimbal_link_roll${self}"/>
-      <origin rpy="0 0 0" xyz="0 0 0"/>
-      <axis xyz="1 0 0"/>
-      <dynamics damping="0.8" friction="0.0"/>
-    </joint>
-    #### gimbal joint (pitch) ####
-    <joint name="gimbal${self}_pitch" type="revolute">
-      <limit effort="6.6" lower="-2.0" upper="2.0" velocity="3.0"/>
-      <parent link="gimbal_link_roll${self}"/>
-      <child link="gimbal_link_pitch${self}"/>
-      <origin rpy="0 0 ${pi/2}" xyz="0.0835 -0.0835 0"/>
-      <axis xyz="1 0 0"/>
-      <dynamics damping="0.8" friction="0.0"/>
-    </joint>
-    <transmission name="joint_tran_roll${self}">
-      <type>transmission_interface/SimpleTransmission</type>
-      <joint name="gimbal${self}_roll">
-        <hardwareInterface>hardware_interface/EffortJointInterface</hardwareInterface>
-      </joint>
-      <actuator name="gimbal${self}_roll_servo">
-        <hardwareInterface>hardware_interface/EffortJointInterface</hardwareInterface>
-        <mechanicalReduction>1</mechanicalReduction>
-      </actuator>
-    </transmission>
-    <transmission name="joint_tran${self}">
-      <type>transmission_integrface/SimpleTransmission</type>
-      <joint name="gimbal${self}_pitch">
-        <hardwareInterface>hardware_interface/EffortJointInterface</hardwareInterface>
-      </joint>
-      <actuator name="gimbal${self}_pitch_servo">
-        <hardwareInterface>hardware_interface/EffortJointInterface</hardwareInterface>
-        <mechanicalReduction>1</mechanicalReduction>
-      </actuator>
-    </transmission>
-    #### rotor parent link joint (virtual) ####
-    <joint name="rotor_parent_link_joint${self}" type="fixed">
-      <parent link="gimbal_link_pitch${self}"/>
-      <child link="rotor_parent${self}"/>
-      <origin rpy="0 0 0" xyz="0.0835 0 0"/>
-      <axis xyz="0 0 ${rotor_direction}"/>
-    </joint>
     #### rotor joint (virtual) ####
     <joint name="rotor${self}" type="continuous">
@@ -226,5 +280,5 @@
       <parent link="rotor_parent${self}"/>
       <child link="thrust${self}"/>
-      <origin rpy="0 0 0" xyz="0 0 0"/>
+      <origin rpy="0 0 0" xyz="0 -0.088 0.02"/>
       <axis xyz="0 0 ${rotor_direction}"/>
     </joint>

File: robots/gimbalrotor/urdf/ynltilt/gimbalrotor.urdf.xacro (robot description, xacro)
@@ -2,4 +2,6 @@
 <robot
     xmlns:xacro="http://www.ros.org/wiki/xacro" name="gimbalrotor_link" >
+  <!-- Include ZED camera macro -->
+  <xacro:include filename="zed_macro.urdf.xacro" />
   <xacro:macro name="gimbalrotor_center_link" params="child1 child2 child3 child4">
     ## dummy
@@ -22,11 +24,42 @@
     ## link
     <link name="base_link">
-      <inertial>
-        <origin xyz="0.001 0.00007 0.00275" rpy="0 0 0"/>
-        <mass value="0.958"/>
-        <inertia
-            ixx="0.01097918" iyy="0.01101753" izz="0.01953502"
-            ixy="-0.00000048" ixz="0.0000" iyz="0.00000"/>
-      </inertial>
+      <!-- Inertial must be calculate in COG and multiple 10^9 against SolidWorks output -->
+    <!--With Pruning-Tool-Sector and zedXmini ON THE PLATE-->
+      <!-- <inertial>
+            <origin xyz="0.06310 -0.00517 0.05062" rpy="0 0 0"/>
+            <mass value="2.33579"/>
+            <inertia
+                ixx="0.03008400484" ixy="-0.00297777401" ixz="-0.00664821011"
+                iyx="-0.00297777401" iyy="0.06882060466" iyz="0.00047002139"
+                izx="-0.00664821011" izy="0.00047002139" izz="0.08922548478"/>
+      </inertial> -->
+      <!--with Pruning-Tool-Sector and zedXmini BETWEEN PLATES-->
+<!--      <inertial>
+        <origin xyz="0.06353 -0.00527 0.04362" rpy="0 0 0"/>
+        <mass value="2.32375"/>
+        <inertia
+            ixx="0.03008400484" ixy="-0.00297777401" ixz="-0.00664821011"
+            iyx="-0.00297777401" iyy="0.06882060466" iyz="0.00047002139"
+            izx="-0.00664821011" izy="0.00047002139" izz="0.08922548478"/>
+	    </inertial>
+-->
+      <!-- Simplest Configuration -->
+      <inertial>
+        <origin xyz="0.00009021 -0.00005299 0.04639014" rpy="0 0 0"/>
+        <mass value="1.16544411"/>
+        <inertia
+            ixx="0.01251517" iyy="0.01254829" izz="0.01920936"
+            ixy="-0.00000046" ixz="-0.00000278" iyz="-0.00001104"/>
+	    </inertial>
+      <!--With Prunning Tools-->
+      <!-- <inertial>
+        <origin xyz="0.05984 0.00138 0.03247" rpy="0 0 0"/>
+        <mass value="1.43147"/>
+        <inertia
+            ixx="0.01393149076" ixy="0.00059865083" ixz="-0.00538129912"
+            iyx="-0.00059865083" iyy="0.03783180404" iyz="-0.00018635030"
+            izx="-0.00538129912" izy="-0.00018635030" izz="0.04319444852"/>
+	</inertial>
+      -->
       <visual>
         <origin xyz="0 0 -0.0" rpy="0 0 0"/>
@@ -125,4 +158,9 @@
     </joint>
     <xacro:friction self="base_link"/>
+    <!-- ZED X MINI Camera Integration -->
+    <xacro:zed_camera name="zedxm" model="zedxm" parent="base_link">
+      <!-- ドローン原点からzedXminiのねじ穴までの相対座標（ZED on TOP plate）-->
+      <origin xyz="0.08653 0.0 0.09595" rpy="0 0 0" />
+    </xacro:zed_camera>
   </xacro:macro>
   <xacro:macro name="gimbalrotor_thrust_link" params="self rotor_direction">
@@ -131,10 +169,10 @@
     <link name="gimbal_link${self}">
       <inertial>
-        <origin xyz="0.018 0.00 0.00438" rpy="0 0 0"/>
-        <mass value="0.1095"/>
-        <inertia
-            ixx="0.00002989" ixy="0.0000"     ixz="-0.0000"
-                             iyy="0.00002848" iyz="0.00000"
-                                              izz="0.0002698"
+        <origin xyz="0.0412 0.00 0.0184" rpy="0 0 0"/>
+        <mass value="0.14"/>
+        <inertia
+            ixx="0.00003614" ixy="0.0000"     ixz="0.00000471"
+                             iyy="0.00004251" iyz="0.00000"
+                                              izz="0.00002946"
         />
       </inertial>
@@ -241,7 +279,8 @@
   </xacro:macro>
   <xacro:extra_module name = "lidar_imu" parent = "base_link" visible = "0" > <!-- should be IMU frame -->
-    <origin xyz="${0.0} ${0.0} ${0.145}" rpy="0 0 ${-pi/2.0}"/> <!-- TODO: the true pos -->
+    <!-- <origin xyz="${0.0} ${0.0} ${0.16082}" rpy="0 0 ${-pi/2.0}"/>  -->
+   <origin xyz="${0.005255} ${-0.004071} ${0.1163}" rpy="0 0 ${-pi/2.0}"/>  <!-- True IMU frame by CAD and validated by calibration -->
     <inertial>
-      <mass value = "00" />
+      <mass value = "0" />
       <origin xyz="0 0 0" rpy="0 0 0"/>
       <inertia
@@ -250,3 +289,32 @@
     </inertial>
   </xacro:extra_module>
+    <!-- Arm (Scissors) rotation center -->
+  <xacro:extra_module name="scissor_center" parent="base_link" visible="1">
+    <origin xyz="0.42126 -0.0154 -0.0003" rpy="0 0 0"/>
+    <inertial>
+      <mass value="0.00001"/>
+      <origin xyz="0 0 0" rpy="0 0 0"/>
+      <inertia
+          ixx="0.000001" ixy="0.0" ixz="0.0"
+          iyy="0.000001" iyz="0.0" izz="0.000001"/>
+    </inertial>
+  </xacro:extra_module>
+  <link name="arm_link_1">
+    <inertial>
+      <mass value="0.001"/>
+      <origin xyz="0 0 0" rpy="0 0 0"/>
+      <inertia ixx="1e-6" ixy="0" ixz="0" iyy="1e-6" iyz="0" izz="1e-6"/>
+    </inertial>
+    <visual>
+      <origin xyz="0 0 0" rpy="0 0 0"/>
+      <geometry>
+        <box size="0.02 0.02 0.02"/>
+      </geometry>
+    </visual>
+  </link>
+  <joint name="scissor_joint" type="fixed">
+    <parent link="scissor_center"/>
+    <child link="arm_link_1"/>
+    <origin xyz="0 0 0" rpy="0 0 0"/>
+  </joint>
 </robot>
