Commit message: zdup, yaw pd up each x1.5

File: robots/gimbalrotor/urdf/ynltilt/gimbalrotor.urdf.xacro (robot description, xacro)
@@ -45,5 +45,5 @@
 -->
       <!-- Simplest Configuration -->
-      <inertial>
+     <!-- <inertial>
         <origin xyz="0.00009021 -0.00005299 0.04639014" rpy="0 0 0"/>
         <mass value="1.16544411"/>
@@ -52,6 +52,7 @@
             ixy="-0.00000046" ixz="-0.00000278" iyz="-0.00001104"/>
 	    </inertial>
+     -->
       <!--With Prunning Tools-->
-      <!-- <inertial>
+      <inertial>
         <origin xyz="0.05984 0.00138 0.03247" rpy="0 0 0"/>
         <mass value="1.43147"/>
@@ -61,5 +62,4 @@
             izx="-0.00538129912" izy="-0.00018635030" izz="0.04319444852"/>
 	</inertial>
-      -->
       <visual>
         <origin xyz="0 0 -0.0" rpy="0 0 0"/>

Commit message: change URDF for zedxm&pruning-sector

File: robots/gimbalrotor/urdf/ynltilt/gimbalrotor.urdf.xacro (robot description, xacro)
@@ -26,5 +26,5 @@
       <!-- Inertial must be calculate in COG and multiple 10^9 against SolidWorks output -->
     <!--With Pruning-Tool-Sector and zedXmini ON THE PLATE-->
-      <!-- <inertial>
+    <inertial>
             <origin xyz="0.06310 -0.00517 0.05062" rpy="0 0 0"/>
             <mass value="2.33579"/>
@@ -33,5 +33,5 @@
                 iyx="-0.00297777401" iyy="0.06882060466" iyz="0.00047002139"
                 izx="-0.00664821011" izy="0.00047002139" izz="0.08922548478"/>
-      </inertial> -->
+      </inertial>
       <!--with Pruning-Tool-Sector and zedXmini BETWEEN PLATES-->
 <!--      <inertial>
@@ -54,5 +54,5 @@
      -->
       <!--With Prunning Tools-->
-      <inertial>
+<!--      <inertial>
         <origin xyz="0.05984 0.00138 0.03247" rpy="0 0 0"/>
         <mass value="1.43147"/>
@@ -62,4 +62,5 @@
             izx="-0.00538129912" izy="-0.00018635030" izz="0.04319444852"/>
 	</inertial>
+-->
       <visual>
         <origin xyz="0 0 -0.0" rpy="0 0 0"/>

Commit message: pushing the changes

File: robots/gimbalrotor/urdf/ynltilt/gimbalrotor.urdf.xacro (robot description, xacro)
@@ -281,5 +281,5 @@
   <xacro:extra_module name = "lidar_imu" parent = "base_link" visible = "0" > <!-- should be IMU frame -->
     <!-- <origin xyz="${0.0} ${0.0} ${0.16082}" rpy="0 0 ${-pi/2.0}"/>  -->
-   <origin xyz="${0.005255} ${-0.004071} ${0.1163}" rpy="0 0 ${-pi/2.0}"/>  <!-- True IMU frame by CAD and validated by calibration -->
+   <origin xyz="${0.005255} ${-0.004071} ${0.11163}" rpy="0 0 ${-pi/2.0}"/>  <!-- True IMU frame by CAD and validated by calibration -->
     <inertial>
       <mass value = "0" />

Commit message: [URDF] calibrate the position of ZEDxMini

File: robots/gimbalrotor/urdf/ynltilt/gimbalrotor.urdf.xacro (robot description, xacro)
@@ -162,5 +162,6 @@
     <xacro:zed_camera name="zedxm" model="zedxm" parent="base_link">
       <!-- ドローン原点からzedXminiのねじ穴までの相対座標（ZED on TOP plate）-->
-      <origin xyz="0.08653 0.0 0.09595" rpy="0 0 0" />
+      <!-- <origin xyz="0.08653 0.0 0.09595" rpy="0 0 0" /> -->
+      <origin xyz="0.089457 0.006355 0.104867" rpy="-0.00410719 -0.00016010 0.01163528" /> <!-- calibrated by LiDAR and ZEDxMini, 2026/6/5 -->
     </xacro:zed_camera>
   </xacro:macro>

Commit message: update camera extrinsic: apply 0614 calibration and comment out 0605

File: robots/gimbalrotor/urdf/ynltilt/gimbalrotor.urdf.xacro (robot description, xacro)
@@ -163,5 +163,6 @@
       <!-- ドローン原点からzedXminiのねじ穴までの相対座標（ZED on TOP plate）-->
       <!-- <origin xyz="0.08653 0.0 0.09595" rpy="0 0 0" /> -->
-      <origin xyz="0.089457 0.006355 0.104867" rpy="-0.00410719 -0.00016010 0.01163528" /> <!-- calibrated by LiDAR and ZEDxMini, 2026/6/5 -->
+      <!-- <origin xyz="0.089457 0.006355 0.104867" rpy="-0.00410719 -0.00016010 0.01163528" /> --> <!-- calibrated by LiDAR and ZEDxMini, 2026/6/5 -->
+      <origin xyz="0.087170 0.000816 0.106766" rpy="-0.01722208 0.00012408 0.01513776" /> <!-- calibrated by LiDAR and ZEDxMini, 2026/6/14 -->
     </xacro:zed_camera>
   </xacro:macro>

Commit message: update zed_camera origin using 0614 merged calibration results

File: robots/gimbalrotor/urdf/ynltilt/gimbalrotor.urdf.xacro (robot description, xacro)
@@ -164,5 +164,5 @@
       <!-- <origin xyz="0.08653 0.0 0.09595" rpy="0 0 0" /> -->
       <!-- <origin xyz="0.089457 0.006355 0.104867" rpy="-0.00410719 -0.00016010 0.01163528" /> --> <!-- calibrated by LiDAR and ZEDxMini, 2026/6/5 -->
-      <origin xyz="0.087170 0.000816 0.106766" rpy="-0.01722208 0.00012408 0.01513776" /> <!-- calibrated by LiDAR and ZEDxMini, 2026/6/14 -->
+      <origin xyz="0.087365 -0.000370 0.100222" rpy="-0.01462965 -0.00390974 0.01466164" /> <!-- calibrated by LiDAR and ZEDxMini, 2026/6/15 (0614 merged) -->
     </xacro:zed_camera>
   </xacro:macro>
